Commit message: reversed changes on xacro file

File: src/gear_place_description/urdf/gear_fr3.urdf.xacro (robot description, xacro)
@@ -3,8 +3,8 @@
   <xacro:arg name="camera" default="true"/>
   <!-- Inclue macros -->
-  <xacro:include filename="$(find franka_description)/robots/fr3_arm.xacro"/>
+  <xacro:include filename="$(find franka_description)/robots/panda_arm.xacro"/>
   <xacro:include filename="$(find franka_description)/robots/hand.xacro"/>
   <xacro:include filename="$(find realsense2_description)/urdf/_d435.urdf.xacro" />
-  <xacro:include filename="$(find franka_description)/robots/fr3_arm.ros2_control.xacro"/>
+  <xacro:include filename="$(find franka_description)/robots/panda_arm.ros2_control.xacro"/>
   <material name="Black">
     <color rgba="${50/255} ${50/255} ${50/255} 1.0"/>
@@ -13,7 +13,7 @@
     <color rgba="${200/255} ${200/255} ${200/255} 1.0"/>
   </material>
-  <!-- Run fr3 macro -->
-  <xacro:fr3_arm
-    arm_id="fr3"
+  <!-- Run panda macro -->
+  <xacro:panda_arm
+    arm_id="panda"
     safety_distance="0.0"
     connected_to="cart_link"
@@ -21,7 +21,7 @@
   <!-- Run hand macro -->
   <xacro:hand
-    ns="fr3"
+    ns="panda"
     rpy="0 0 ${-pi/4}"
-    connected_to="fr3_link8"
+    connected_to="panda_link8"
     safety_distance="0.0"/>
   <!-- Joints -->
@@ -46,5 +46,5 @@
     <joint name="camera_mount_to_flange_joint" type="fixed">
       <origin xyz="0.03 0 .045" rpy="0 0 0"/>
-      <parent link="fr3_hand"/>
+      <parent link="panda_hand"/>
       <child link="camera_mount" />
     </joint>
@@ -64,6 +64,6 @@
   </xacro:if>
   <!-- Run ROS2 control macro -->
-  <xacro:fr3_arm_ros2_control
-    ns="fr3"
+  <xacro:panda_arm_ros2_control
+    ns="panda"
     robot_ip="172.16.0.2"
     use_fake_hardware="false"

Commit message: updates

File: src/gear_place_description/urdf/gear_fr3.urdf.xacro (robot description, xacro)
@@ -3,8 +3,7 @@
   <xacro:arg name="camera" default="true"/>
   <!-- Inclue macros -->
-  <xacro:include filename="$(find franka_description)/robots/panda_arm.xacro"/>
-  <xacro:include filename="$(find franka_description)/robots/hand.xacro"/>
+  <xacro:include filename="$(find gear_place_description)/robots/common/franka_arm.xacro"/>
+  <xacro:include filename="$(find gear_place_description)/robots/common/franka_hand.xacro"/>
   <xacro:include filename="$(find realsense2_description)/urdf/_d435.urdf.xacro" />
-  <xacro:include filename="$(find franka_description)/robots/panda_arm.ros2_control.xacro"/>
   <material name="Black">
     <color rgba="${50/255} ${50/255} ${50/255} 1.0"/>
@@ -13,19 +12,25 @@
     <color rgba="${200/255} ${200/255} ${200/255} 1.0"/>
   </material>
+  <link name="world"/>
+  <link name="cart_link"/>
   <!-- Run panda macro -->
-  <xacro:panda_arm
-    arm_id="panda"
+  <xacro:franka_arm
+    arm_id="fr3"
+    connected_to="cart_link"
+    xyz="0.05 0.0 0.0"
+    joint_limits="${xacro.load_yaml('$(find gear_place_description)/urdf/joint_limits.yaml')}"
+    description_pkg="gear_place_description"/>
+  <!-- Run hand macro -->
+  <xacro:franka_hand
+    arm_id="fr3"
+    rpy="0 0 ${-pi/4}"
+    tcp_xyz="0 0 0.1034"
+    tcp_rpy="0 0 0"
+    connected_to="fr3_link8"
     safety_distance="0.0"
-    connected_to="cart_link"
-    xyz="0.05 0 0"/>
-  <!-- Run hand macro -->
-  <xacro:hand
-    ns="panda"
-    rpy="0 0 ${-pi/4}"
-    connected_to="panda_link8"
-    safety_distance="0.0"/>
+    description_pkg="gear_place_description"/>
   <!-- Joints -->
   <joint name="cart_to_world" type="fixed">
-    <origin xyz="-0.3945 0.55 0.0127" rpy="0 0 0"/>
+    <origin xyz="0 0 0.5" rpy="0 0 0"/>
     <parent link="world"/>
     <child link="cart_link" />
@@ -46,5 +51,5 @@
     <joint name="camera_mount_to_flange_joint" type="fixed">
       <origin xyz="0.03 0 .045" rpy="0 0 0"/>
-      <parent link="panda_hand"/>
+      <parent link="fr3_hand"/>
       <child link="camera_mount" />
     </joint>
@@ -63,9 +68,3 @@
     </xacro:sensor_d435>
   </xacro:if>
-  <!-- Run ROS2 control macro -->
-  <xacro:panda_arm_ros2_control
-    ns="panda"
-    robot_ip="172.16.0.2"
-    use_fake_hardware="false"
-    fake_sensor_commands="false"/>
 </robot>
